File: Electric_Water_Heater/Schema&Layout/Electric_Water_Heater.kicad_sch (KiCad schematic)
At the start: 26 parts, among them J1 Barrel_Jack_Switch, SW1 SW_Push, U1 ATmega32A-P, U2 L7805, U3 7447, U4 ELD-426SYGWA, U5 ST24C08, Y1 16MHz

Commit message: Update_Schematic
Parts:
- added C6, C7: 0.1uF, symbol Device:C
- added D3: LED, symbol Device:LED
- added D4: 1N4007, Diode_THT:D_DO-41_SOD81_P10.16mm_Horizontal, symbol Diode:1N4007
- added J2: Conn_01x08_Pin, symbol Connector:Conn_01x08_Pin
- added J3, J4: Screw_Terminal_01x02, symbol Connector:Screw_Terminal_01x02
- added K1: JQC-3FF-005-1Z, Relay_THT:Relay_SPDT_Hongfa_JQC-3FF_0XX-1Z, symbol Relay:JQC-3FF-005-1Z
- added R12: 330, symbol Device:R
- C2: value 1uF -> 0.1uF
Connections:
- net +5V: now also U1.30 (AVCC), C6.1, C7.1
- net GND: now also C6.2, C7.2, D3.1 (K), D4.2 (A), K1.12, K1.A2
- net PD5: now reaches U1.19 (PD5)
- net PD5: now also R12.2
- net PC2: now reaches U1.24 (PC2)
- net PC2: now also D4.1 (K), K1.A1
- new net: D3.2 (A), R12.1
Other:
- moved on the sheet: D2, R1
